File: mmdvm_hs_dual_hat.kicad_pcb (KiCad board)
At the start: 2 copper layers, 65 x 56 mm, 119 parts, among them J1 RPi_GPIO, P1 SMA, P2 SMA, P25 red, P3 I2C, P4 DISPLAY, P5 STLINK, P6 USB_OTG, P7 CONN_02X03, SW1 DNI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

Commit message: add holes and more GND on PCB
Routing:
- net GND: vias 3 -> 21
Changed lines of the file:
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@@
     (thickness 1.6)
     (drawings 27)
-    (tracks 1302)
+    (tracks 1324)
     (zones 0)
     (modules 119)
@@
     (0 F.Cu signal hide)
     (31 B.Cu signal hide)
-    (32 B.Adhes user hide)
+    (32 B.Adhes user)
     (33 F.Adhes user hide)
     (34 B.Paste user)
-    (35 F.Paste user hide)
-    (36 B.SilkS user hide)
+    (35 F.Paste user)
+    (36 B.SilkS user)
     (37 F.SilkS user)
     (38 B.Mask user hide)
@@
     (pad_to_mask_clearance 0)
     (aux_axis_origin 0 0)
-    (visible_elements 7FEFA461)
+    (visible_elements 7EFEA22F)
     (pcbplotparams
       (layerselection 0x010f0_ffffffff)
@@
   (gr_line (start 93.25 138.5) (end 152.25 138.5) (angle 90) (layer Edge.Cuts) (width 0.1))
   (gr_line (start 155.25 85.5) (end 155.25 135.5) (angle 90) (layer Edge.Cuts) (width 0.1))
+  (via (at 113.7 104) (size 0.6) (drill 0.4) (layers F.Cu B.Cu) (net 3))
+  (via (at 115 104) (size 0.6) (drill 0.4) (layers F.Cu B.Cu) (net 3))
+  (via (at 116.3 104) (size 0.6) (drill 0.4) (layers F.Cu B.Cu) (net 3))
+  (via (at 116.3 102.7) (size 0.6) (drill 0.4) (layers F.Cu B.Cu) (net 3))
+  (via (at 116.3 105.3) (size 0.6) (drill 0.4) (layers F.Cu B.Cu) (net 3))
+  (via (at 115 105.3) (size 0.6) (drill 0.4) (layers F.Cu B.Cu) (net 3))
+  (via (at 113.7 105.3) (size 0.6) (drill 0.4) (layers F.Cu B.Cu) (net 3))
+  (via (at 115 102.7) (size 0.6) (drill 0.4) (layers F.Cu B.Cu) (net 3))
+  (via (at 113.7 102.7) (size 0.6) (drill 0.4) (layers F.Cu B.Cu) (net 3))
+  (via (at 113.9 129.1) (size 0.6) (drill 0.4) (layers F.Cu B.Cu) (net 3))
+  (via (at 115.2 129.1) (size 0.6) (drill 0.4) (layers F.Cu B.Cu) (net 3))
+  (via (at 116.5 129.1) (size 0.6) (drill 0.4) (layers F.Cu B.Cu) (net 3))
+  (via (at 116.5 127.8) (size 0.6) (drill 0.4) (layers F.Cu B.Cu) (net 3))
+  (via (at 115.2 127.8) (size 0.6) (drill 0.4) (layers F.Cu B.Cu) (net 3))
+  (via (at 113.9 127.8) (size 0.6) (drill 0.4) (layers F.Cu B.Cu) (net 3))
+  (via (at 116.5 126.5) (size 0.6) (drill 0.4) (layers F.Cu B.Cu) (net 3))
+  (via (at 115.2 126.5) (size 0.6) (drill 0.4) (layers F.Cu B.Cu) (net 3))
+  (via (at 113.9 126.5) (size 0.6) (drill 0.4) (layers F.Cu B.Cu) (net 3))
   (segment (start 144.52 84.76) (end 143.3311 84.76) (width 0.25) (layer F.Cu) (net 1) (status 10))
   (segment (start 141.45 102) (end 141.45 102.6253) (width 0.25) (layer F.Cu) (net 1) (status 10))
@@
   (segment (start 141.317 129.8417) (end 152.5204 129.8417) (width 0.25) (layer F.Cu) (net 33))
   (segment (start 139.6753 128.2) (end 141.317 129.8417) (width 0.25) (layer F.Cu) (net 33))
+  (segment (start 113.013346 100.97031) (end 115.447756 100.97031) (width 0.25) (layer B.Cu) (net 34))
+  (segment (start 115.447756 100.97031) (end 116.25 100.168066) (width 0.25) (layer B.Cu) (net 34))
+  (segment (start 111.3356 102.648056) (end 113.013346 100.97031) (width 0.25) (layer B.Cu) (net 34))
+  (segment (start 111.3356 103.8759) (end 111.3356 102.648056) (width 0.25) (layer B.Cu) (net 34))
+  (segment (start 119.9551 103.873166) (end 116.25 100.168066) (width 0.25) (layer B.Cu) (net 34))
+  (segment (start 116.25 100.168066) (end 116.25 98.6683) (width 0.25) (layer B.Cu) (net 34))
+  (segment (start 119.9551 103.8759) (end 119.9551 103.873166) (width 0.25) (layer B.Cu) (net 34))
   (via (at 109.016 130.81) (size 0.6) (layers F.Cu B.Cu) (net 34))
   (via (at 109.9615 105.25) (size 0.6) (layers F.Cu B.Cu) (net 34))
@@
   (segment (start 143.6611 128.05) (end 140.5308 124.9197) (width 0.25) (layer F.Cu) (net 34))
   (segment (start 116.25 98.6683) (end 116.25 100.6) (width 0.25) (layer F.Cu) (net 34) (status 20))
-  (segment (start 116.25 103.8759) (end 116.25 98.6683) (width 0.25) (layer B.Cu) (net 34))
-  (segment (start 111.3356 103.8759) (end 116.25 103.8759) (width 0.25) (layer B.Cu) (net 34))
   (segment (start 119.9551 103.8759) (end 120.4592 104.38) (width 0.25) (layer B.Cu) (net 34))
-  (segment (start 116.25 103.8759) (end 119.9551 103.8759) (width 0.25) (layer B.Cu) (net 34))
   (segment (start 129.3772 100.4247) (end 129.5 100.4247) (width 0.25) (layer F.Cu) (net 34))
   (segment (start 129.0109 100.0584) (end 129.3772 100.4247) (width 0.25) (layer F.Cu) (net 34))
@@
     (polygon
       (pts
-        (xy 90.2 82.5) (xy 155.2 82.5) (xy 155.2 138.5) (xy 90.3 138.5)
+        (xy 90 82.4) (xy 155.6 82.4) (xy 155.4 138.6) (xy 90 138.6)
       )
     )
